File: Breadboard_Power_Supply/Breadboard_Power_Supply.kicad_pcb (KiCad board)
At the start: 2 copper layers, 32.3 x 55.8 mm, 19 parts, among them J1 Barrel_Jack, J3 Conn_01x02_Pin, J4 Conn_01x02_Pin, J5 Conn_01x03_Pin, J6 Screw_Terminal_01x02, J7 Conn_01x03_Pin, J8 Screw_Terminal_01x02, SW1 SW_Wuerth_450301014042, U1 LM7805_TO220, U2 LM317_TO-220

Commit message: Breadboard_Power_Supply_V2
Parts:
- J1: value Barrel_Jack -> Barrel_Jack_Switch
Connections:
- J3 pad 2: /PWR_OUTPUT -> /PWR_OUTPUT_TOP
- J4 pad 2: /PWR_OUTPUT -> /PWR_OUTPUT_BOT
- J5 pad 2: /PWR_OUTPUT -> /PWR_OUTPUT_TOP
- J6 pad 1: /PWR_OUTPUT -> /PWR_OUTPUT_TOP
- J7 pad 2: /PWR_OUTPUT -> /PWR_OUTPUT_BOT
- J8 pad 1: /PWR_OUTPUT -> /PWR_OUTPUT_BOT
Routing:
- net /PWR_OUTPUT: track 114.8 -> 0.00 mm
- net /PWR_OUTPUT_BOT: track 0.00 -> 26.6 mm
- net /PWR_OUTPUT_TOP: track 0.00 -> 23.9 mm
Changed lines of the file:
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@@
 	)
 	(paper "A4")
+	(title_block
+		(title "Breadboard_Power_Supply_Layout")
+		(date "2026-02-03")
+		(rev "2")
+	)
 	(layers
 		(0 "F.Cu" signal)
@@
 	(net 6 "Net-(D2-A)")
 	(net 7 "/PWR_INPUT")
-	(net 8 "/PWR_OUTPUT")
+	(net 8 "/PWR_OUTPUT_TOP")
 	(net 9 "Net-(U2-ADJ)")
 	(net 10 "unconnected-(SW1-C-Pad2)")
+	(net 11 "/PWR_OUTPUT_BOT")
 	(footprint "Resistor_THT:R_Axial_DIN0204_L3.6mm_D1.6mm_P7.62mm_Horizontal"
 		(layer "F.Cu")
@@
 		(property ki_fp_filters "R_*")
 		(sheetname "/")
-		(sheetfile "Simple_Power_Supply.kicad_sch")
+		(sheetfile "Breadboard_Power_Supply.kicad_sch")
 		(attr through_hole)
 		(fp_line
@@
 		(property ki_fp_filters "TO-???* *_Diode_* *SingleDiode* D_*")
 		(sheetname "/")
-		(sheetfile "Simple_Power_Supply.kicad_sch")
+		(sheetfile "Breadboard_Power_Supply.kicad_sch")
 		(attr through_hole)
 		(fp_line
@@
 		(property ki_fp_filters "C_*")
 		(sheetname "/")
-		(sheetfile "Simple_Power_Supply.kicad_sch")
+		(sheetfile "Breadboard_Power_Supply.kicad_sch")
 		(attr through_hole)
 		(fp_line
@@
 		(property ki_fp_filters "C_*")
 		(sheetname "/")
-		(sheetfile "Simple_Power_Supply.kicad_sch")
+		(sheetfile "Breadboard_Power_Supply.kicad_sch")
 		(attr through_hole)
 		(fp_line
@@
 		(property ki_fp_filters "Connector*:*_1x??_*")
 		(sheetname "/")
-		(sheetfile "Simple_Power_Supply.kicad_sch")
+		(sheetfile "Breadboard_Power_Supply.kicad_sch")
 		(attr through_hole)
 		(fp_line
@@
 			(layers "*.Cu" "*.Mask")
 			(remove_unused_layers no)
-			(net 8 "/PWR_OUTPUT")
+			(net 11 "/PWR_OUTPUT_BOT")
 			(pinfunction "Pin_2")
 			(pintype "passive")
@@
 		(property ki_fp_filters "Connector*:*_1x??_*")
 		(sheetname "/")
-		(sheetfile "Simple_Power_Supply.kicad_sch")
+		(sheetfile "Breadboard_Power_Supply.kicad_sch")
 		(attr through_hole)
 		(fp_line
@@
 			(layers "*.Cu" "*.Mask")
 			(remove_unused_layers no)
-			(net 8 "/PWR_OUTPUT")
+			(net 8 "/PWR_OUTPUT_TOP")
 			(pinfunction "Pin_2")
 			(pintype "passive")
@@
 		(property ki_fp_filters "C_*")
 		(sheetname "/")
-		(sheetfile "Simple_Power_Supply.kicad_sch")
+		(sheetfile "Breadboard_Power_Supply.kicad_sch")
 		(attr through_hole)
 		(fp_line
@@
 		(property ki_fp_filters "SW*Wuerth*WS*SLTV*10x2.5x6.4*P2.54mm*")
 		(sheetname "/")
-		(sheetfile "Simple_Power_Supply.kicad_sch")
+		(sheetfile "Breadboard_Power_Supply.kicad_sch")
 		(attr through_hole)
 		(fp_rect
@@
 		(property ki_fp_filters "TO?220*")
 		(sheetname "/")
-		(sheetfile "Simple_Power_Supply.kicad_sch")
+		(sheetfile "Breadboard_Power_Supply.kicad_sch")
 		(attr through_hole)
 		(fp_line
@@
 			)
 		)
-		(property "Value" "Barrel_Jack"
+		(property "Value" "Barrel_Jack_Switch"
 			(at -6.4928 -5.5 0)
 			(layer "F.SilkS")
@@
 		(property ki_fp_filters "BarrelJack*")
 		(sheetname "/")
-		(sheetfile "Simple_Power_Supply.kicad_sch")
+		(sheetfile "Breadboard_Power_Supply.kicad_sch")
 		(attr through_hole)
 		(fp_line
@@
 		(property ki_fp_filters "C_*")
 		(sheetname "/")
-		(sheetfile "Simple_Power_Supply.kicad_sch")
+		(sheetfile "Breadboard_Power_Supply.kicad_sch")
 		(attr through_hole)
 		(fp_line
@@
 		(property ki_fp_filters "R_*")
 		(sheetname "/")
-		(sheetfile "Simple_Power_Supply.kicad_sch")
+		(sheetfile "Breadboard_Power_Supply.kicad_sch")
 		(attr through_hole)
 		(fp_line
@@
 		(property ki_fp_filters "TerminalBlock*:*")
 		(sheetname "/")
-		(sheetfile "Simple_Power_Supply.kicad_sch")
+		(sheetfile "Breadboard_Power_Supply.kicad_sch")
 		(attr through_hole)
 		(fp_line
@@
 			(remove_unused_layers no)
 			(roundrect_rratio 0.096154)
-			(net 8 "/PWR_OUTPUT")
+			(net 11 "/PWR_OUTPUT_BOT")
 			(pinfunction "Pin_1")
 			(pintype "passive")
@@
 		(property ki_fp_filters "Connector*:*_1x??_*")
 		(sheetname "/")
-		(sheetfile "Simple_Power_Supply.kicad_sch")
+		(sheetfile "Breadboard_Power_Supply.kicad_sch")
 		(attr through_hole)
 		(fp_line
@@
 			(layers "*.Cu" "*.Mask")
 			(remove_unused_layers no)
-			(net 8 "/PWR_OUTPUT")
+			(net 11 "/PWR_OUTPUT_BOT")
 			(pinfunction "Pin_2")
 			(pintype "passive")
@@
 		(property ki_fp_filters "Connector*:*_1x??_*")
 		(sheetname "/")
-		(sheetfile "Simple_Power_Supply.kicad_sch")
+		(sheetfile "Breadboard_Power_Supply.kicad_sch")
 		(attr through_hole)
 		(fp_line
@@
 			(layers "*.Cu" "*.Mask")
 			(remove_unused_layers no)
-			(net 8 "/PWR_OUTPUT")
+			(net 8 "/PWR_OUTPUT_TOP")
 			(pinfunction "Pin_2")
 			(pintype "passive")
@@
 		(property ki_fp_filters "TO?220*")
 		(sheetname "/")
-		(sheetfile "Simple_Power_Supply.kicad_sch")
+		(sheetfile "Breadboard_Power_Supply.kicad_sch")
 		(attr through_hole)
 		(fp_line
@@
 		(property ki_fp_filters "LED* LED_SMD:* LED_THT:*")
 		(sheetname "/")
-		(sheetfile "Simple_Power_Supply.kicad_sch")
+		(sheetfile "Breadboard_Power_Supply.kicad_sch")
 		(attr through_hole)
 		(fp_line
@@
 		(property ki_fp_filters "R_*")
 		(sheetname "/")
-		(sheetfile "Simple_Power_Supply.kicad_sch")
+		(sheetfile "Breadboard_Power_Supply.kicad_sch")
 		(attr through_hole)
 		(fp_line
@@
 		(property ki_fp_filters "TerminalBlock*:*")
 		(sheetname "/")
-		(sheetfile "Simple_Power_Supply.kicad_sch")
+		(sheetfile "Breadboard_Power_Supply.kicad_sch")
 		(attr through_hole)
 		(fp_line
@@
 			(remove_unused_layers no)
 			(roundrect_rratio 0.096154)
-			(net 8 "/PWR_OUTPUT")
+			(net 8 "/PWR_OUTPUT_TOP")
 			(pinfunction "Pin_1")
 			(pintype "passive")
@@
 	)
 	(segment
-		(start 118.33837 109.524)
-		(end 123.1908 109.524)
-		(width 0.35)
-		(layer "F.Cu")
-		(net 8)
-	)
-	(segment
 		(start 117.015 57.0775)
-		(end 118.3165 55.776)
+		(end 118.291 55.8015)
 		(width 0.35)
 		(layer "F.Cu")
@@
 	)
 	(segment
-		(start 125.8824 71.755)
-		(end 121.4374 71.755)
+		(start 137.0552 59.5834)
+		(end 136.0342 60.6044)
 		(width 0.35)
 		(layer "F.Cu")
@@
 	)
 	(segment
-		(start 130.51 62.3268)
+		(start 125.7071 55.8015)
 		(end 130.51 60.6044)
 		(width 0.35)
@@
 	)
 	(segment
-		(start 126.356 104.5665)
-		(end 125.51 104.5665)
-		(width 0.35)
-		(layer "F.Cu")
-		(net 8)
-	)
-	(segment
-		(start 118.3165 55.776)
-		(end 128.6994 55.776)
-		(width 0.35)
-		(layer "F.Cu")
-		(net 8)
-	)
-	(segment
-		(start 137.0552 59.5834)
-		(end 136.0342 60.6044)
-		(width 0.35)
-		(layer "F.Cu")
-		(net 8)
-	)
-	(segment
-		(start 123.1908 109.524)
-		(end 125.51 107.2048)
-		(width 0.35)
-		(layer "F.Cu")
-		(net 8)
-	)
-	(segment
-		(start 133.1722 97.7503)
-		(end 133.1722 79.0448)
-		(width 0.35)
-		(layer "F.Cu")
-		(net 8)
-	)
-	(segment
-		(start 119.7356 70.0532)
-		(end 119.7356 68.072)
-		(width 0.35)
-		(layer "F.Cu")
-		(net 8)
-	)
-	(segment
-		(start 129.4473 108.5038)
-		(end 125.51 104.5665)
-		(width 0.35)
-		(layer "F.Cu")
-		(net 8)
-	)
-	(segment
-		(start 125.51 107.2048)
-		(end 125.51 104.5665)
-		(width 0.35)
-		(layer "F.Cu")
-		(net 8)
-	)
-	(segment
-		(start 133.1722 97.7503)
-		(end 126.356 104.5665)
-		(width 0.35)
-		(layer "F.Cu")
-		(net 8)
-	)
-	(segment
-		(start 119.7356 68.072)
-		(end 121.5898 66.2178)
-		(width 0.35)
-		(layer "F.Cu")
-		(net 8)
-	)
-	(segment
-		(start 137.0838 108.5038)
-		(end 129.4473 108.5038)
+		(start 118.291 55.8015)
+		(end 125.7071 55.8015)
 		(width 0.35)
 		(layer "F.Cu")
@@
 	)
 	(segment
-		(start 130.51 57.5866)
-		(end 130.51 60.6044)
-		(width 0.35)
-		(layer "F.Cu")
-		(net 8)
-	)
-	(segment
-		(start 133.1722 79.0448)
-		(end 125.8824 71.755)
-		(width 0.35)
-		(layer "F.Cu")
-		(net 8)
-	)
-	(segment
-		(start 117.015 108.20063)
-		(end 118.33837 109.524)
-		(width 0.35)
-		(layer "F.Cu")
-		(net 8)
-	)
-	(segment
-		(start 128.6994 55.776)
-		(end 130.51 57.5866)
-		(width 0.35)
-		(layer "F.Cu")
-		(net 8)
-	)
-	(segment
-		(start 121.4374 71.755)
-		(end 119.7356 70.0532)
-		(width 0.35)
-		(layer "F.Cu")
-		(net 8)
-	)
-	(segment
-		(start 121.5898 66.2178)
-		(end 126.619 66.2178)
-		(width 0.35)
-		(layer "F.Cu")
-		(net 8)
-	)
-	(segment
-		(start 126.619 66.2178)
-		(end 130.51 62.3268)
-		(width 0.35)
-		(layer "F.Cu")
-		(net 8)
-	)
-	(segment
 		(start 131.51 91)
 		(end 129.8254 92.6846)
@@
 		(net 9)
 	)
+	(segment
+		(start 137.0838 108.5038)
+		(end 129.4473 108.5038)
+		(width 0.35)
+		(layer "F.Cu")
+		(net 11)
+	)
+	(segment
+		(start 126.356 104.5665)
+		(end 125.51 104.5665)
+		(width 0.35)
+		(layer "F.Cu")
+		(net 11)
+	)
+	(segment
+		(start 125.51 106.76)
+		(end 125.51 104.5665)
+		(width 0.35)
+		(layer "F.Cu")
+		(net 11)
+	)
+	(segment
+		(start 122.53 109.74)
+		(end 125.51 106.76)
+		(width 0.35)
+		(layer "F.Cu")
+		(net 11)
+	)
+	(segment
+		(start 117.015 108.20063)
+		(end 118.55437 109.74)
+		(width 0.35)
+		(layer "F.Cu")
+		(net 11)
+	)
+	(segment
+		(start 118.55437 109.74)
+		(end 122.53 109.74)
+		(width 0.35)
+		(layer "F.Cu")
+		(net 11)
+	)
+	(segment
+		(start 129.4473 108.5038)
+		(end 125.51 104.5665)
+		(width 0.35)
+		(layer "F.Cu")
+		(net 11)
+	)
 	(zone
