File: Breadboard_Power_Supply/Breadboard_Power_Supply.kicad_sch (KiCad schematic)
At the start: 19 parts, among them J1 Barrel_Jack_Switch, J3 Conn_01x02_Pin, J4 Conn_01x02_Pin, J5 Conn_01x03_Pin, J6 Screw_Terminal_01x02, J7 Conn_01x03_Pin, J8 Screw_Terminal_01x02, SW1 SW_Wuerth_450301014042, U1 LM7805_TO220, U2 LM317_TO-220

Commit message: Breadboard_Power_Supply_V2
Connections:
- net PWR_OUTPUT renamed PWR_OUTPUT_BOT
- net PWR_OUTPUT_BOT: no longer J3.2 (Pin_2), J5.2 (Pin_2), J6.1 (Pin_1)
- new net PWR_OUTPUT_TOP: J3.2 (Pin_2), J5.2 (Pin_2), J6.1 (Pin_1)
Other:
- title: Simple_Power_Supply -> Simple_Power_Supply_Schema
Changed lines of the file:
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@@
 	(paper "A4")
 	(title_block
-		(title "Simple_Power_Supply")
-		(date "2026-01-30")
-		(rev "1")
+		(title "Simple_Power_Supply_Schema")
+		(date "2026-02-03")
+		(rev "2")
 	)
 	(rectangle
@@
 		)
 	)
-	(label "PWR_OUTPUT"
+	(label "PWR_OUTPUT_TOP"
 		(at 186.69 63.5 0)
 		(effects
@@
 		)
 	)
-	(label "PWR_OUTPUT"
+	(label "PWR_OUTPUT_BOT"
 		(at 186.69 107.95 0)
 		(effects
