File: ESP 8266_Dev_Board/ESP 8266_Dev_Board/esp 8266 dev board.kicad_pcb (KiCad board)
At the start: 2 copper layers, 79 x 30.5 mm, 28 parts, among them J1 USB_C_Receptacle_USB2.0_16P, J3 Conn_01x06_Pin, J4 Conn_01x06_Pin, J5 Conn_01x05_Pin, SW2 SW_SPST, SW3 SW_SPST, U1 AMS1117-3.3, U3 CH340C, U4 ESP8266-12E_ESP-12E

Commit message: README File Added
Parts:
- removed hole_1, hole_2, hole_3, hole_4: MountingHole_3mm_Pad, MountingHole:MountingHole_3mm_Pad
- added REF**: MountingHole_2.5mm_Pad, MountingHole:MountingHole_2.5mm_Pad, F.Cu at (151.7, 76.0)
- added REF**: MountingHole_2.5mm_Pad, MountingHole:MountingHole_2.5mm_Pad, F.Cu at (79.7, 100.0)
- added REF**: MountingHole_2.5mm_Pad, MountingHole:MountingHole_2.5mm_Pad, F.Cu at (151.7, 100.0)
- added REF**: MountingHole_2.5mm_Pad, MountingHole:MountingHole_2.5mm_Pad, F.Cu at (79.7, 76.0)
- moved C5 4.87 mm to (100.6, 89.5), turned to 180 degrees
- moved D3 3.78 mm to (120.5, 92.5), turned to 90 degrees
- moved C4 1.01 mm to (110.4, 92.7), turned to 90 degrees
- moved SW2 0.52 mm to (123.7, 98.0)
- moved R3 0.38 mm to (127.6, 97.5)
Routing:
- net GND: track 0.00 -> 36.3 mm
- net Net-(D2-A): track 24.8 -> 29.9 mm
- net Net-(D3-A): track 2.90 -> 5.52 mm
- net D-: track 29.8 -> 32.0 mm
- net SCK: track 21.5 -> 22.8 mm
- net REST: track 46.4 -> 45.4 mm
- net DTR: track 20.2 -> 19.7 mm
- removed copper zone on B.Cu, net GND
