File: Dual Force Plate/Dual Force Plate/Dual Force Plate.kicad_sch (KiCad schematic)
At the start: 22 parts, among them J10 Conn_01x07_Pin, J3 Conn_01x07_Pin, J4 Conn_01x07_Pin, J6 Conn_01x02_Pin, J7 Conn_01x04_Pin, J8 Conn_01x02_Pin, J9 Conn_01x07_Pin, SW1 SW_SPST, U1 MT3608, U2 ESP32-DevKitC, U3 HX711_ADC_24-Bit, U4 HX711_ADC_24-Bit, U5 HX711_ADC_24-Bit, U6 HX711_ADC_24-Bit, U7 TP4056_Dev_Board

Commit message: Final Edit on Mixed Signal Board
Other:
- company: (none) -> Mo3_Tech
Changed lines of the file:
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@@
 		(date "2026-05-06")
 		(rev "1")
+		(company "Mo3_Tech")
 	)
 	(rectangle
